File: hw/a500kbd.kicad_sch (KiCad schematic)
At the start: 17 parts, among them J1 SERIAL, J2 AVR-ISP-6, J3 ps2ribbon, J4 ps2ribbon, SW1 SW_DPDT_x2, U1 ATmega88-20P, U2 intkbd, U3 ps2conn, U4 kbout, Y1 14.7456MHz

Commit message: fixed mirrored ps2 connector in schematic
Connections:
- net GND: now also U3.3 (GND); no longer U3.4 (VCC)
- net PCLK: now also U3.5 (CLK); no longer U3.1 (DATA)
- net PDATA: now also U3.1 (DATA); no longer U3.5 (CLK)
- net VCC: now also U3.4 (VCC); no longer U3.3 (GND)
Other:
- moved on the sheet: U3
Changed lines of the file:
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@@
 	(symbol
 		(lib_id "a500kbd:ps2conn")
-		(at 95.25 77.47 90)
+		(at 95.25 77.47 270)
+		(mirror x)
 		(unit 1)
 		(exclude_from_sim no)
@@
 		(dnp no)
 		(property "Reference" "U3"
-			(at 88.9 83.312 0)
+			(at 101.6 83.312 0)
 			(effects
 				(font
@@
 		)
 		(property "Footprint" "a500kbd:minidin6"
-			(at 113.538 78.994 0)
+			(at 76.962 78.994 0)
 			(effects
 				(font

Commit message: fixed pcb, ps/2 connector facing the wrong way
Parts:
- C1, C2: footprint Capacitor_THT:C_Disc_D3.0mm_W2.0mm_P2.50mm -> Capacitor_THT:C_Disc_D4.3mm_W1.9mm_P5.00mm
- U4: footprint Connector_PinHeader_2.54mm:PinHeader_1x08_P2.54mm_Vertical -> Connector_PinSocket_2.54mm:PinSocket_1x08_P2.54mm_Vertical
Changed lines of the file:
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@@
 (kicad_sch
-	(version 20231120)
+	(version 20250114)
 	(generator "eeschema")
-	(generator_version "8.0")
+	(generator_version "9.0")
 	(paper "A5" portrait)
 	(title_block
@@
 		(comment 2 "Copyright (C) 2017-2025 John Tsiombikas <nuclear@mutantstargoat.com>")
 	)
+	(text "Optional ribbon cable end points\nfor break-away PS/2 connector board"
+		(exclude_from_sim no)
+		(at 113.03 32.766 0)
+		(effects
+			(font
+				(size 1.27 1.27)
+			)
+		)
+	)
 	(junction
 		(at 71.12 124.46)
@@
 		)
 	)
-	(text "Optional ribbon cable end points\nfor break-away PS/2 connector board"
-		(exclude_from_sim no)
-		(at 113.03 32.766 0)
-		(effects
-			(font
-				(size 1.27 1.27)
-			)
-		)
-	)
 	(label "PDATA"
 		(at 118.11 52.07 0)
-		(fields_autoplaced yes)
 		(effects
 			(font
@@
 	(label "PCLK"
 		(at 118.11 58.42 0)
-		(fields_autoplaced yes)
 		(effects
 			(font
@@
 	(label "ACLK"
 		(at 46.99 92.71 0)
-		(fields_autoplaced yes)
 		(effects
 			(font
@@
 	(label "TXD"
 		(at 68.58 87.63 0)
-		(fields_autoplaced yes)
 		(effects
 			(font
@@
 	(label "ADATA"
 		(at 46.99 97.79 0)
-		(fields_autoplaced yes)
 		(effects
 			(font
@@
 	(label "XTAL1"
 		(at 44.45 59.69 0)
-		(fields_autoplaced yes)
 		(effects
 			(font
@@
 	(label "~{RESET}"
 		(at 49.53 80.01 0)
-		(fields_autoplaced yes)
 		(effects
 			(font
@@
 	(label "MOSI"
 		(at 45.72 49.53 0)
-		(fields_autoplaced yes)
 		(effects
 			(font
@@
 	(label "SCK"
 		(at 45.72 54.61 0)
-		(fields_autoplaced yes)
 		(effects
 			(font
@@
 	(label "AMIGA_RESET"
 		(at 76.2 137.16 0)
-		(fields_autoplaced yes)
 		(effects
 			(font
@@
 	(label "RXD"
 		(at 68.58 85.09 0)
-		(fields_autoplaced yes)
 		(effects
 			(font
@@
 	(label "PDATA"
 		(at 46.99 95.25 0)
-		(fields_autoplaced yes)
 		(effects
 			(font
@@
 	(label "PCLK"
 		(at 118.11 49.53 0)
-		(fields_autoplaced yes)
 		(effects
 			(font
@@
 	(label "ODAT"
 		(at 105.41 105.41 0)
-		(fields_autoplaced yes)
 		(effects
 			(font
@@
 	(label "OCLK"
 		(at 105.41 115.57 0)
-		(fields_autoplaced yes)
 		(effects
 			(font
@@
 	(label "INTKB_DATA"
 		(at 68.58 111.76 0)
-		(fields_autoplaced yes)
 		(effects
 			(font
@@
 	(label "XTAL0"
 		(at 44.45 57.15 0)
-		(fields_autoplaced yes)
 		(effects
 			(font
@@
 	(label "MISO"
 		(at 45.72 52.07 0)
-		(fields_autoplaced yes)
 		(effects
 			(font
@@
 	(label "PCLK"
 		(at 46.99 90.17 0)
-		(fields_autoplaced yes)
 		(effects
 			(font
@@
 	(label "STLED"
 		(at 78.74 121.92 0)
-		(fields_autoplaced yes)
 		(effects
 			(font
@@
 	(label "DRVLED"
 		(at 78.74 124.46 0)
-		(fields_autoplaced yes)
 		(effects
 			(font
@@
 	(label "PDATA"
 		(at 118.11 60.96 0)
-		(fields_autoplaced yes)
 		(effects
 			(font
@@
 	(label "INTKB_CLOCK"
 		(at 68.58 114.3 0)
-		(fields_autoplaced yes)
 		(effects
 			(font
@@
 			)
 		)
-		(property "Description" "1x8 pin header 2.54mm female"
+		(property "Description" "1x8 pin header 2.54mm male"
 			(at 55.88 116.84 0)
 			(effects
@@
 			)
 		)
-		(property "Datasheet" " ~"
+		(property "Datasheet" "~"
 			(at 114.935 66.04 0)
 			(effects
@@
 			)
 		)
-		(property "Footprint" "Connector_PinHeader_2.54mm:PinHeader_1x08_P2.54mm_Vertical"
+		(property "Footprint" "Connector_PinSocket_2.54mm:PinSocket_1x08_P2.54mm_Vertical"
 			(at 135.89 133.35 0)
 			(effects
@@
 			)
 		)
-		(property "Description" "1x8 pin header 2.54mm male"
+		(property "Description" "1x8 pin header 2.54mm female"
 			(at 128.27 116.84 0)
 			(effects
@@
 			)
 		)
-		(property "Footprint" "Capacitor_THT:C_Disc_D3.0mm_W2.0mm_P2.50mm"
+		(property "Footprint" "Capacitor_THT:C_Disc_D4.3mm_W1.9mm_P5.00mm"
 			(at 25.0952 138.43 0)
 			(effects
@@
 			)
 		)
-		(property "Footprint" "Capacitor_THT:C_Disc_D3.0mm_W2.0mm_P2.50mm"
+		(property "Footprint" "Capacitor_THT:C_Disc_D4.3mm_W1.9mm_P5.00mm"
 			(at 32.7152 138.43 0)
 			(effects
@@
 		)
 	)
+	(embedded_fonts no)
 )
